File: hardware/project-stemmaqt-ds2482.sch (KiCad schematic (older format))
At the start: 1 part

Commit message: First draft
Parts:
- added C?: 100nF, Capacitor_SMD:C_0603_1608Metric, symbol Device:C
- added D?: LED, LED_SMD:LED_0603_1608Metric, symbol Device:LED
- added H? (x4): MountingHole_Pad, MountingHole:MountingHole_2.2mm_M2_Pad, symbol Mechanical:MountingHole_Pad
- added J? (x2): SM04B-SRSS-TB(LF)(SN), JST_SM04B-SRSS-TB(LF)(SN), symbol SM04B-SRSS-TB_LF__SN_:SM04B-SRSS-TB(LF)(SN)
- added J? (x2): Conn_01x03_Male, Connector_PinHeader_2.54mm:PinHeader_1x03_P2.54mm_Vertical, symbol Connector:Conn_01x03_Male
- added JP? (x3): SolderJumper_2_Open, Jumper:SolderJumper-2_P1.3mm_Open_RoundedPad1.0x1.5mm, symbol Jumper:SolderJumper_2_Open
- added Q?: Q_PMOS_GSD, Package_TO_SOT_SMD:SOT-23, symbol Device:Q_PMOS_GSD
- added R? (x5): 10k, Resistor_SMD:R_0603_1608Metric, symbol Device:R
- added R?: SPU, Resistor_SMD:R_0603_1608Metric, symbol Device:R
Connections:
- net labels added: 1WIRE, GND, PCTLZ, SCL, SDA, VCC
- wire segments 0 -> 66
Other:
- moved on the sheet: U?

Commit message: Schematic annotation
Parts:
- gave numbers to parts that had none: 21
Changed lines of the file:
@@
 $EndDescr
 $Comp
-L DS2482S-100_:DS2482S-100+ U?
+L DS2482S-100_:DS2482S-100+ U1
 U 1 1 612ED155
 P 2300 3650
-F 0 "U?" H 2300 4217 50  0000 C CNN
+F 0 "U1" H 2300 4217 50  0000 C CNN
 F 1 "DS2482S-100+" H 2300 4126 50  0000 C CNN
 F 2 "SOIC127P600X175-8N" H 2300 3650 50  0001 L BNN
@@
 $EndComp
 $Comp
-L Device:R R?
+L Device:R R1
 U 1 1 612F35A0
 P 1000 4050
-F 0 "R?" H 1070 4096 50  0000 L CNN
+F 0 "R1" H 1070 4096 50  0000 L CNN
 F 1 "10k" H 1070 4005 50  0000 L CNN
 F 2 "Resistor_SMD:R_0603_1608Metric" V 930 4050 50  0001 C CNN
@@
 $EndComp
 $Comp
-L Device:R R?
+L Device:R R2
 U 1 1 612F3DA9
 P 1300 4050
-F 0 "R?" H 1370 4096 50  0000 L CNN
+F 0 "R2" H 1370 4096 50  0000 L CNN
 F 1 "10k" H 1370 4005 50  0000 L CNN
 F 2 "Resistor_SMD:R_0603_1608Metric" V 1230 4050 50  0001 C CNN
@@
 	1300 3650 1600 3650
 $Comp
-L Jumper:SolderJumper_2_Open JP?
+L Jumper:SolderJumper_2_Open JP1
 U 1 1 612FA65D
 P 1000 3250
-F 0 "JP?" V 1000 3318 50  0000 L CNN
+F 0 "JP1" V 1000 3318 50  0000 L CNN
 F 1 "SolderJumper_2_Open" V 1045 3318 50  0001 L CNN
 F 2 "Jumper:SolderJumper-2_P1.3mm_Open_RoundedPad1.0x1.5mm" H 1000 3250 50  0001 C CNN
@@
 $EndComp
 $Comp
-L Jumper:SolderJumper_2_Open JP?
+L Jumper:SolderJumper_2_Open JP2
 U 1 1 612FBECB
 P 1300 3250
-F 0 "JP?" V 1300 3318 50  0000 L CNN
+F 0 "JP2" V 1300 3318 50  0000 L CNN
 F 1 "SolderJumper_2_Open" V 1345 3318 50  0001 L CNN
 F 2 "Jumper:SolderJumper-2_P1.3mm_Open_RoundedPad1.0x1.5mm" H 1300 3250 50  0001 C CNN
@@
 	1000 3550 1000 3900
 $Comp
-L Device:R R?
+L Device:R R4
 U 1 1 612FFFBC
 P 3300 3100
-F 0 "R?" H 3370 3146 50  0000 L CNN
+F 0 "R4" H 3370 3146 50  0000 L CNN
 F 1 "10k" H 3370 3055 50  0000 L CNN
 F 2 "Resistor_SMD:R_0603_1608Metric" V 3230 3100 50  0001 C CNN
@@
 $EndComp
 $Comp
-L Device:R R?
+L Device:R R5
 U 1 1 6130064E
 P 3600 3100
-F 0 "R?" H 3670 3146 50  0000 L CNN
+F 0 "R5" H 3670 3146 50  0000 L CNN
 F 1 "10k" H 3670 3055 50  0000 L CNN
 F 2 "Resistor_SMD:R_0603_1608Metric" V 3530 3100 50  0001 C CNN
@@
 	3100 3950 3000 3950
 $Comp
-L Device:C C?
+L Device:C C1
 U 1 1 61314C76
 P 1000 1300
-F 0 "C?" H 1115 1346 50  0000 L CNN
+F 0 "C1" H 1115 1346 50  0000 L CNN
 F 1 "100nF" H 1115 1255 50  0000 L CNN
 F 2 "Capacitor_SMD:C_0603_1608Metric" H 1000 1300 50  0001 C CNN
@@
 1WIRE
 $Comp
-L Jumper:SolderJumper_2_Open JP?
+L Jumper:SolderJumper_2_Open JP3
 U 1 1 6132B4E0
 P 5300 3850
-F 0 "JP?" V 5300 3918 50  0000 L CNN
+F 0 "JP3" V 5300 3918 50  0000 L CNN
 F 1 "SolderJumper_2_Open" V 5345 3918 50  0001 L CNN
 F 2 "Jumper:SolderJumper-2_P1.3mm_Open_RoundedPad1.0x1.5mm" H 5300 3850 50  0001 C CNN
@@
 	5300 4100 5850 4100
 $Comp
-L Device:R R?
+L Device:R R6
 U 1 1 6134763A
 P 5300 2950
-F 0 "R?" H 5370 2996 50  0000 L CNN
+F 0 "R6" H 5370 2996 50  0000 L CNN
 F 1 "SPU" H 5370 2905 50  0000 L CNN
 F 2 "Resistor_SMD:R_0603_1608Metric" V 5230 2950 50  0001 C CNN
@@
 	1000 1600 1000 1650
 $Comp
-L Device:Q_PMOS_GSD Q?
+L Device:Q_PMOS_GSD Q1
 U 1 1 613716E7
 P 5200 3400
-F 0 "Q?" H 5405 3354 50  0000 L CNN
+F 0 "Q1" H 5405 3354 50  0000 L CNN
 F 1 "Q_PMOS_GSD" H 5405 3445 50  0000 L CNN
 F 2 "Package_TO_SOT_SMD:SOT-23" H 5400 3500 50  0001 C CNN
@@
 $EndComp
 $Comp
-L SM04B-SRSS-TB_LF__SN_:SM04B-SRSS-TB(LF)(SN) J?
+L SM04B-SRSS-TB_LF__SN_:SM04B-SRSS-TB(LF)(SN) J1
 U 1 1 6137759C
 P 3550 1100
-F 0 "J?" H 3550 1450 50  0000 C CNN
+F 0 "J1" H 3550 1450 50  0000 C CNN
 F 1 "SM04B-SRSS-TB(LF)(SN)" H 3493 1476 50  0001 C CNN
 F 2 "JST_SM04B-SRSS-TB(LF)(SN)" H 3550 1100 50  0001 L BNN
@@
 $EndComp
 $Comp
-L SM04B-SRSS-TB_LF__SN_:SM04B-SRSS-TB(LF)(SN) J?
+L SM04B-SRSS-TB_LF__SN_:SM04B-SRSS-TB(LF)(SN) J2
 U 1 1 6137B0FC
 P 4650 1100
-F 0 "J?" H 4600 1450 50  0000 L CNN
+F 0 "J2" H 4600 1450 50  0000 L CNN
 F 1 "SM04B-SRSS-TB(LF)(SN)" H 4593 624 50  0001 C CNN
 F 2 "JST_SM04B-SRSS-TB(LF)(SN)" H 4650 1100 50  0001 L BNN
@@
 	4350 1400 3950 1400
 $Comp
-L power:GND #PWR?
+L power:GND #PWR03
 U 1 1 6138D126
 P 3950 1500
-F 0 "#PWR?" H 3950 1250 50  0001 C CNN
+F 0 "#PWR03" H 3950 1250 50  0001 C CNN
 F 1 "GND" H 3955 1327 50  0000 C CNN
 F 2 "" H 3950 1500 50  0001 C CNN
@@
 GND
 $Comp
-L power:VCC #PWR?
+L power:VCC #PWR01
 U 1 1 613AB82B
 P 2100 950
-F 0 "#PWR?" H 2100 800 50  0001 C CNN
+F 0 "#PWR01" H 2100 800 50  0001 C CNN
 F 1 "VCC" H 2115 1123 50  0000 C CNN
 F 2 "" H 2100 950 50  0001 C CNN
@@
 $EndComp
 $Comp
-L power:GND #PWR?
+L power:GND #PWR02
 U 1 1 613ABDDB
 P 2100 1750
-F 0 "#PWR?" H 2100 1500 50  0001 C CNN
+F 0 "#PWR02" H 2100 1500 50  0001 C CNN
 F 1 "GND" H 2105 1577 50  0000 C CNN
 F 2 "" H 2100 1750 50  0001 C CNN
@@
 $EndComp
 $Comp
-L Device:R R?
+L Device:R R3
 U 1 1 613ACADC
 P 2100 1150
-F 0 "R?" H 2170 1196 50  0000 L CNN
+F 0 "R3" H 2170 1196 50  0000 L CNN
 F 1 "10k" H 2170 1105 50  0000 L CNN
 F 2 "Resistor_SMD:R_0603_1608Metric" V 2030 1150 50  0001 C CNN
@@
 $EndComp
 $Comp
-L Device:LED D?
+L Device:LED D1
 U 1 1 613B255F
 P 2100 1500
-F 0 "D?" V 2093 1382 50  0000 R CNN
+F 0 "D1" V 2093 1382 50  0000 R CNN
 F 1 "LED" V 2055 1430 50  0001 R CNN
 F 2 "LED_SMD:LED_0603_1608Metric" V 2100 1500 50  0001 C CNN
@@
 	2100 1650 2100 1750
 $Comp
-L Connector:Conn_01x03_Male J?
+L Connector:Conn_01x03_Male J3
 U 1 1 613DEF1D
 P 5500 950
-F 0 "J?" H 5550 1150 50  0000 C CNN
+F 0 "J3" H 5550 1150 50  0000 C CNN
 F 1 "Conn_01x03_Male" H 5608 1140 50  0001 C CNN
 F 2 "Connector_PinHeader_2.54mm:PinHeader_1x03_P2.54mm_Vertical" H 5500 950 50  0001 C CNN
@@
 VCC
 $Comp
-L Connector:Conn_01x03_Male J?
+L Connector:Conn_01x03_Male J4
 U 1 1 613EDDA6
 P 6150 950
-F 0 "J?" H 6200 1150 50  0000 C CNN
+F 0 "J4" H 6200 1150 50  0000 C CNN
 F 1 "Conn_01x03_Male" H 6258 1140 50  0001 C CNN
 F 2 "Connector_PinHeader_2.54mm:PinHeader_1x03_P2.54mm_Vertical" H 6150 950 50  0001 C CNN
@@
 VCC
 $Comp
-L Mechanical:MountingHole_Pad H?
+L Mechanical:MountingHole_Pad H1
 U 1 1 613F9A62
 P 7400 950
-F 0 "H?" H 7500 953 50  0000 L CNN
+F 0 "H1" H 7500 953 50  0000 L CNN
 F 1 "MountingHole_Pad" H 7500 908 50  0001 L CNN
 F 2 "MountingHole:MountingHole_2.2mm_M2_Pad" H 7400 950 50  0001 C CNN
@@
 $EndComp
 $Comp
-L Mechanical:MountingHole_Pad H?
+L Mechanical:MountingHole_Pad H2
 U 1 1 613FBBE3
 P 7700 950
-F 0 "H?" H 7800 953 50  0000 L CNN
+F 0 "H2" H 7800 953 50  0000 L CNN
 F 1 "MountingHole_Pad" H 7800 908 50  0001 L CNN
 F 2 "MountingHole:MountingHole_2.2mm_M2_Pad" H 7700 950 50  0001 C CNN
@@
 $EndComp
 $Comp
-L Mechanical:MountingHole_Pad H?
+L Mechanical:MountingHole_Pad H3
 U 1 1 613FBE9D
 P 8000 950
-F 0 "H?" H 8100 953 50  0000 L CNN
+F 0 "H3" H 8100 953 50  0000 L CNN
 F 1 "MountingHole_Pad" H 8100 908 50  0001 L CNN
 F 2 "MountingHole:MountingHole_2.2mm_M2_Pad" H 8000 950 50  0001 C CNN
@@
 $EndComp
 $Comp
-L Mechanical:MountingHole_Pad H?
+L Mechanical:MountingHole_Pad H4
 U 1 1 613FC1ED
 P 8300 950
-F 0 "H?" H 8400 953 50  0000 L CNN
+F 0 "H4" H 8400 953 50  0000 L CNN
 F 1 "MountingHole_Pad" H 8400 908 50  0001 L CNN
 F 2 "MountingHole:MountingHole_2.2mm_M2_Pad" H 8300 950 50  0001 C CNN
@@
 $EndComp
 $Comp
-L power:GND #PWR?
+L power:GND #PWR04
 U 1 1 613FCD2C
 P 7400 1250
-F 0 "#PWR?" H 7400 1000 50  0001 C CNN
+F 0 "#PWR04" H 7400 1000 50  0001 C CNN
 F 1 "GND" H 7405 1077 50  0000 C CNN
 F 2 "" H 7400 1250 50  0001 C CNN

Commit message: Little schematic cleanup
Parts:
- added C?: 10uF, Capacitor_SMD:C_1210_3225Metric, symbol Device:C
Connections:
- wire segments 66 -> 68
Other:
- note added: "Connectors"
- note added: "Decoupling"
- note added: "LED"
- note added: "Mounting"
- moved on the sheet: C1, D1, H1, H2, H3, H4, J1, J2, J3, J4, R3

Commit message: Annotation
Parts:
- gave numbers to parts that had none: 1
Changed lines of the file:
@@
 $EndComp
 $Comp
-L Device:C C?
+L Device:C C2
 U 1 1 6145671A
 P 1650 1350
-F 0 "C?" H 1765 1396 50  0000 L CNN
+F 0 "C2" H 1765 1396 50  0000 L CNN
 F 1 "10uF" H 1765 1305 50  0000 L CNN
 F 2 "Capacitor_SMD:C_1210_3225Metric" H 1650 1350 50  0001 C CNN
@@
 $EndComp
 $Comp
-L power:VCC #PWR?
+L power:VCC #PWR05
 U 1 1 61456720
 P 1650 1000
-F 0 "#PWR?" H 1650 850 50  0001 C CNN
+F 0 "#PWR05" H 1650 850 50  0001 C CNN
 F 1 "VCC" H 1665 1173 50  0000 C CNN
 F 2 "" H 1650 1000 50  0001 C CNN
@@
 $EndComp
 $Comp
-L power:GND #PWR?
+L power:GND #PWR06
 U 1 1 61456726
 P 1650 1700
-F 0 "#PWR?" H 1650 1450 50  0001 C CNN
+F 0 "#PWR06" H 1650 1450 50  0001 C CNN
 F 1 "GND" H 1655 1527 50  0000 C CNN
 F 2 "" H 1650 1700 50  0001 C CNN

Commit message: Placement draft
Parts:
- H1, H2, H3, H4: footprint MountingHole:MountingHole_2.2mm_M2_Pad -> MountingHole:MountingHole_2.2mm_M2_ISO7380_Pad
- JP1: value SolderJumper_2_Open -> AD0
- JP2: value SolderJumper_2_Open -> AD1
- JP3: value SolderJumper_2_Open -> SPU
Changed lines of the file:
@@
 P 1000 3250
 F 0 "JP1" V 1000 3318 50  0000 L CNN
-F 1 "SolderJumper_2_Open" V 1045 3318 50  0001 L CNN
+F 1 "AD0" V 1045 3318 50  0001 L CNN
 F 2 "Jumper:SolderJumper-2_P1.3mm_Open_RoundedPad1.0x1.5mm" H 1000 3250 50  0001 C CNN
 F 3 "~" H 1000 3250 50  0001 C CNN
@@
 P 1300 3250
 F 0 "JP2" V 1300 3318 50  0000 L CNN
-F 1 "SolderJumper_2_Open" V 1345 3318 50  0001 L CNN
+F 1 "AD1" V 1345 3318 50  0001 L CNN
 F 2 "Jumper:SolderJumper-2_P1.3mm_Open_RoundedPad1.0x1.5mm" H 1300 3250 50  0001 C CNN
 F 3 "~" H 1300 3250 50  0001 C CNN
@@
 P 5300 3850
 F 0 "JP3" V 5300 3918 50  0000 L CNN
-F 1 "SolderJumper_2_Open" V 5345 3918 50  0001 L CNN
+F 1 "SPU" V 5345 3918 50  0001 L CNN
 F 2 "Jumper:SolderJumper-2_P1.3mm_Open_RoundedPad1.0x1.5mm" H 5300 3850 50  0001 C CNN
 F 3 "~" H 5300 3850 50  0001 C CNN
@@
 F 0 "H4" H 9300 1153 50  0000 L CNN
 F 1 "MountingHole_Pad" H 9300 1108 50  0001 L CNN
-F 2 "MountingHole:MountingHole_2.2mm_M2_Pad" H 9200 1150 50  0001 C CNN
+F 2 "MountingHole:MountingHole_2.2mm_M2_ISO7380_Pad" H 9200 1150 50  0001 C CNN
 F 3 "~" H 9200 1150 50  0001 C CNN
 	1    9200 1150
@@
 F 0 "H3" H 9000 1153 50  0000 L CNN
 F 1 "MountingHole_Pad" H 9000 1108 50  0001 L CNN
-F 2 "MountingHole:MountingHole_2.2mm_M2_Pad" H 8900 1150 50  0001 C CNN
+F 2 "MountingHole:MountingHole_2.2mm_M2_ISO7380_Pad" H 8900 1150 50  0001 C CNN
 F 3 "~" H 8900 1150 50  0001 C CNN
 	1    8900 1150
@@
 F 0 "H2" H 8700 1153 50  0000 L CNN
 F 1 "MountingHole_Pad" H 8700 1108 50  0001 L CNN
-F 2 "MountingHole:MountingHole_2.2mm_M2_Pad" H 8600 1150 50  0001 C CNN
+F 2 "MountingHole:MountingHole_2.2mm_M2_ISO7380_Pad" H 8600 1150 50  0001 C CNN
 F 3 "~" H 8600 1150 50  0001 C CNN
 	1    8600 1150
@@
 F 0 "H1" H 8400 1153 50  0000 L CNN
 F 1 "MountingHole_Pad" H 8400 1108 50  0001 L CNN
-F 2 "MountingHole:MountingHole_2.2mm_M2_Pad" H 8300 1150 50  0001 C CNN
+F 2 "MountingHole:MountingHole_2.2mm_M2_ISO7380_Pad" H 8300 1150 50  0001 C CNN
 F 3 "~" H 8300 1150 50  0001 C CNN
 	1    8300 1150

Commit message: First placement done
Parts:
- removed J4: Conn_01x03_Male, Connector_PinHeader_2.54mm:PinHeader_1x03_P2.54mm_Vertical, symbol Connector:Conn_01x03_Male
Connections:
- wire segments 68 -> 65
Changed lines of the file:
@@
-	1    0    0    -1
-$EndComp
-Text Label 7050 1050 0    50   ~ 0
-VCC
-Text Label 7050 1150 0    50   ~ 0
-1WIRE
-Text Label 7050 1250 0    50   ~ 0
-GND
-Wire Wire Line
-	7300 1250 7050 1250
-Wire Wire Line
-	7300 1150 7050 1150
-Wire Wire Line
-	7300 1050 7050 1050
-$Comp
-L Connector:Conn_01x03_Male J4
-U 1 1 613EDDA6
-P 6850 1150
-F 0 "J4" H 6900 1350 50  0000 C CNN
-F 1 "Conn_01x03_Male" H 6958 1340 50  0001 C CNN
-F 2 "Connector_PinHeader_2.54mm:PinHeader_1x03_P2.54mm_Vertical" H 6850 1150 50  0001 C CNN
-F 3 "~" H 6850 1150 50  0001 C CNN
-	1    6850 1150
 	1    0    0    -1
 $EndComp
